File: PCB_kicadV5/PGPExT_v1-1.kicad_pcb (KiCad board)
At the start: 4 copper layers, 25.5 x 25.2 mm, 53 parts, among them SW1 SW_SPDT, U1 TS5A3166, U2 TC1271A, U3 SN74AUC1GU, U4 TPS22918, U5 ADG888YRUZ, U6 TPS76930, U7 ATTINY44A-SSU

Commit message: update to 1.1
fixing diode pin assignment and routing
Parts:
- D2, D4: footprint Package_TO_SOT_SMD:SOT-343_SC-70-4 -> additional_parts:SOT-343_4_mod
- turned D4 to 180 degrees
Connections:
- D2 pad 3: Net-(C6-Pad1) -> Net-(D2-Pad3)
- D2 pad 4: Net-(D2-Pad4) -> Net-(C6-Pad1)
- R7 pad 1: Net-(D2-Pad4) -> Net-(D2-Pad3)
Routing:
- net Net-(D4-Pad2): track 2.00 -> 4.43 mm
- net Net-(D2-Pad4): track 1.96 -> 0.00 mm
- net Net-(D2-Pad3): track 0.00 -> 1.96 mm
- net Net-(C7-Pad1): track 4.09 -> 5.79 mm
- net Net-(C6-Pad1): track 4.39 -> 6.08 mm
- net Net-(D2-Pad2): track 1.96 -> 3.17 mm
- net /PGPExt_Signal_Processing/LEDr_i: track 18.7 -> 19.6 mm
Other:
- board text added: "Ext1V1"
- board text removed: "Bugfix: solder W10 = LEDg W16 = LEDb"
- board text removed: "ExtV1"
